File: Hardware/PCB.brd (EAGLE design)
At the start: 170.4 x 111.2 mm, 103 parts, among them IC1 BD5229G-TR, IC4 XC6220A331MR-G, J1 FH34SRJ-24S-0.5SH_99_, J2 SAMACSYS_PARTS_USB4110-GF-A, J3 QWIIC_RIGHT_ANGLE, J4 112A-TAAR-R03_ATTEND, Q1 20V/4.2A/52mΩ/1.4W, Q2 20V/4.2A/52mΩ/1.4W, Q3 SI1308EDL-T1-GE3, U1 W25Q512JVEIQ, U2 ESP32-C6-WROOM-1-N8, U3 DS3231SN#, U4 MAX17048G+T10

Commit message: Add files via upload
Parts:
- R1_PINH1, R2-PINH1: value (none) -> 10K
- moved R_RESET 1.50 mm to (31.0, 111.0)
- moved C6 1.40 mm to (47.0, 111.2)
- moved R_BOOT 1.30 mm to (55.8, 111.2)
- moved C10 1.10 mm to (62.2, 111.1)
- moved C5 0.92 mm to (22.4, 111.3)
- moved R_CHANGE 0.90 mm to (70.5, 111.1)
- renumbered TP1 to TX, TP10 to EPD_CS, TP11 to EPD_DC, TP12 to EPD_RST, TP13 to EPD_3V3_C, TP14 to VBUS, TP15 to INT_RTC, TP16 to 3V3, TP17 to EPD_3V3, TP2 to RX, TP3 to VBAT, TP4 to GND, TP5 to GND-2, TP6 to MISO, TP7 to MOSI, TP8 to SCK, TP9 to EPD_BUSY
Routing:
- net GND: track 0.00 -> 639.4 mm, vias 0 -> 7
- net MOSI: track 0.00 -> 217.2 mm, vias 0 -> 6
- net INT_RTC: track 168.1 -> 138.9 mm
- net EPD_RST: track 180.6 -> 155.6 mm, vias 3 -> 4
- net SRC: track 71.5 -> 49.5 mm, vias 0 -> 2
- net 3V3: track 482.8 -> 499.9 mm, vias 14 -> 12
- net EPD_3V3_C: track 159.6 -> 142.7 mm, vias 3 -> 2
- net EPD_3V3: track 88.2 -> 103.9 mm, vias 6 -> 5
- net DN: track 0.00 -> 13.8 mm
- net DP: track 0.00 -> 13.2 mm
- net EPD_BUSY: track 153.8 -> 144.8 mm, vias 4 -> 5
- net MISO: track 120.6 -> 113.1 mm, vias 5 -> 6
- net N$25: track 26.3 -> 31.1 mm
- net SS_SD: track 98.5 -> 102.4 mm
- net EPD_DC: track 108.4 -> 105.2 mm
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- added copper zone on layer 1, net GND
- added copper zone on layer 16, net GND
